File: ESP32/ESP32.kicad_pcb (KiCad board)
At the start: 2 copper layers, 30 x 30 mm, 65 parts, among them J1 BAT_CON, J2 Conn_Coaxial, J3 Conn_02x10_Odd_Even, J4 Conn_02x10_Odd_Even, P1 USB_C_Plug_USB2.0, Q1 DMG2301L, SW1 SW_SPST, SW2 SW_SPST, U1 TPS63001, U2 MCP73831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

Commit message: Components are organized
Parts:
- removed C6: 10mf, Capacitor_SMD:C_0805_2012Metric
- removed F1: Fuse, Fuse:Fuse_0805_2012Metric_Pad1.15x1.40mm_HandSolder
- added D5: B220, Diode_SMD:D_SOD-323, F.Cu at (112.2, 82.4)
- added F2: Fuse, Fuse:Fuse_0805_2012Metric_Pad1.15x1.40mm_HandSolder, F.Cu at (105.0, 72.0)
- AE1: footprint Johanson:2450AT42A100E -> Antenna:2450AT42A100E
- C1, C2, C4, C5: footprint Capacitor_SMD:C_0805_2012Metric -> Capacitor_SMD:C_0603_1608Metric
- C15: value 10mf -> 1mF
- C3: footprint Capacitor_SMD:C_0805_2012Metric -> Capacitor_SMD:C_0402_1005Metric
- D2: footprint Diode_SMD:D_SMB -> Diode_SMD:D_SOD-323
- J3, J4: footprint footprints:BM28B0.6-20DS&slash_2-0.35V51 -> FPC3:HRS_DF12NB-20DS-0.5V(51); moved to B.Cu
- R10: value 10K -> 2K
- R11: value 10K -> 442K
- R12: value 10K -> 160K
- R9: value 10K -> 3.3K
- Y1: footprint Crystal:Crystal_SMD_0603-4Pin_6.0x3.5mm -> Crystal:Crystal_SMD_3225-4Pin_3.2x2.5mm
- moved J1 180.4 mm to (127.0, 72.8), turned to 90 degrees
- moved Y1 169.4 mm to (121.8, 91.3)
- moved AE1 166.2 mm to (128.3, 96.4), turned to 90 degrees
- moved U4 165.4 mm to (108.0, 95.6)
- moved J4 164.9 mm to (115.2, 94.0), turned to 180 degrees
- moved C10 164.3 mm to (126.2, 86.4)
- moved J3 164.1 mm to (115.2, 75.8), turned to 180 degrees
- moved C16 163.0 mm to (125.5, 95.9), turned to -90 degrees
- moved C12 162.8 mm to (126.2, 85.2)
- moved C11 162.7 mm to (126.2, 82.7)
- moved C17 162.4 mm to (123.6, 95.9), turned to -90 degrees
- moved C13 162.3 mm to (125.2, 88.8)
- moved C15 161.6 mm to (125.2, 90.2)
- moved C14 161.4 mm to (126.2, 83.9)
- moved C22 159.4 mm to (125.0, 92.5), turned to 180 degrees
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Connections:
- C1 pad 1: VCC -> Net-(Q1-S)
- C2 pad 1: VCC -> Net-(Q1-S)
- C4 pad 1: Net-(C4-Pad1) -> +3.3V
- C5 pad 1: Net-(C4-Pad1) -> +3.3V
- D2 pad 1: VCC -> Net-(D2-K)
- Q1 pad 2: VCC -> Net-(Q1-S)
- U1 pad 1: Net-(C4-Pad1) -> +3.3V
- U1 pad 10: Net-(C4-Pad1) -> +3.3V
- U1 pad 10B: Net-(C4-Pad1) -> +3.3V
- U1 pad 1B: Net-(C4-Pad1) -> +3.3V
- U1 pad 5: VCC -> Net-(Q1-S)
- U1 pad 5B: VCC -> Net-(Q1-S)
